File: eagle/tinyled.brd (EAGLE design)
At the start: 32.7 x 29.2 mm, 11 parts, among them IC1 ATtiny85

Commit message: fixed shiort circuits in design
Parts:
- added R4: 10k, eagle-ltspice:0204/7
- moved R3 1.27 mm to (5.08, 7.62)
- moved USER1 1.27 mm to (26.7, 24.1)
Connections:
- net +5V: now also R4.1
- net RESET: now also R4.2
Routing:
- net RESET: track 0.00 -> 23.4 mm
- net +5V: track 26.9 -> 43.4 mm
- net EXTV: track 27.5 -> 22.3 mm
- net SWITCH1: track 10.3 -> 8.98 mm
- net N$1: track 6.15 -> 7.42 mm
- net DATA: track 32.4 -> 33.5 mm
